File: pcb/halo-90.kicad_sch (KiCad schematic)
At the start: 102 parts, among them J1 TC2030-SWIM-NL, U1 STM8151G6U6, U2 SC7A20HTR, U3 DRV5032

Commit message: fix(pcb): update JLCPCB BOM component LCSC parts
- Set BT1 (CR2032 holder) to C70377
- Set U3 (DRV5032) to C130005
- Set D1-D90 (0402 LEDs) to C198650
- Renamed 100n capacitors to 100nF for JLC verification match
- Regenerated BOM and Gerbers archive
Parts:
- C1, C2, C3: value 100n -> 100nF
- U3: LCSC Part# C2655033 -> C130005
Changed lines of the file:
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@@
 			)
 		)
-		(property "Value" "100n"
+		(property "Value" "100nF"
 			(at 223.52 114.2999 0)
 			(effects
@@
 			)
 		)
-		(property "Value" "100n"
+		(property "Value" "100nF"
 			(at 242.57 107.9499 0)
 			(effects
@@
 			)
 		)
-		(property "Value" "100n"
+		(property "Value" "100nF"
 			(at 182.88 52.0699 0)
 			(effects
@@
 			)
 		)
-		(property "LCSC Part#" "C2655033"
+		(property "LCSC Part#" "C130005"
 			(at 257.81 123.19 0)
 			(effects
